File: smol-DAP/smol-DAP.sch (KiCad schematic (older format))
At the start: 4 parts

Commit message: First pass at the smol dap
Parts:
- removed J?: Conn_02x05_Odd_Even, symbol Connector_Generic:Conn_02x05_Odd_Even
- added C1, C4: 1u, Capacitor_SMD:C_0402_1005Metric, symbol Device:C_Small
- added C10, C9: 22p, Capacitor_SMD:C_0402_1005Metric, symbol Device:C_Small
- added C2, C3, C5, C6, C7, C8: 100n, Capacitor_SMD:C_0402_1005Metric, symbol Device:C_Small
- added D1: GREEN, LED_SMD:LED_0603_1608Metric, symbol Device:LED_ALT
- added D2: BLUE, LED_SMD:LED_0603_1608Metric, symbol Device:LED_ALT
- added D3: RED, LED_SMD:LED_0603_1608Metric, symbol Device:LED_ALT
- added J2: Conn_ARM_JTAG_SWD_10, Connector:Tag-Connect_TC2050-IDC-NL_2x05_P1.27mm_Vertical, symbol Connector:Conn_ARM_JTAG_SWD_10
- added R1, R2: 22R, Resistor_SMD:R_0402_1005Metric, symbol Device:R_Small_US
- added R10, R9: 4.7k, Resistor_SMD:R_0402_1005Metric, symbol Device:R_Small_US
- added R11, R6, R7: 10k, Resistor_SMD:R_0402_1005Metric, symbol Device:R_Small_US
- added R3: 100R, Resistor_SMD:R_0402_1005Metric, symbol Device:R_Small_US
- added R4, R5, R8: 470, Resistor_SMD:R_0402_1005Metric, symbol Device:R_Small_US
- added U1: AP2127K-3.3, Package_TO_SOT_SMD:SOT-23-5, symbol Regulator_Linear:AP2127K-3.3
- added Y1: 8MHz, Crystal:Crystal_SMD_Abracon_ABM8G-4Pin_3.2x2.5mm, symbol Device:Crystal_GND24_Small
- J1: renamed from J?; footprint (none) -> Connector_USB:USB_C_Receptacle_GCT_USB4085
- J3: renamed from J?; footprint (none) -> Connector_PinHeader_1.00mm:PinHeader_2x05_P1.00mm_Vertical_SMD
- gave numbers to parts that had none: 1
Connections:
- net +3V3: now also C3.1, C4.1, C5.1, C6.1, C7.1, C8.1, D1.2 (A), D2.2 (A), J2.1 (VTref), R11.2, R9.2, U1.5 (VOUT)
- net GND: now also J1.A1 (GND), J1.A12 (GND), J1.B1 (GND), J1.B12 (GND), J1.S1 (SHIELD), J3.3 (Pin_3), J3.5 (Pin_5), U2.20 (PB2), C1.2, C10.2, C2.2, C3.2, C4.2, C5.2, C6.2, C7.2, C8.2, C9.1, D3.1 (K), J2.3 (GND), J2.5 (GND), J2.9 (GNDDetect), R10.1, R6.2, R7.2, U1.2 (GND), Y1.2, Y1.4
- net SWCLK: now also J2.4 (SWDCLK/TCK)
- net SWDIO: now also J2.2 (SWDIO/TMS)
- net ~RESET: now also J2.10 (~RESET~), R11.1
- net at U2.10 (PA0): now also R10.2, R9.1
- net TGT_RX: now reaches U2.12 (PA2)
- net TGT_RX: now also J3.7 (Pin_7)
- net TGT_TX: now reaches U2.13 (PA3)
- net TGT_TX: now also J3.9 (Pin_9)
- net TGT_SWCLK: now reaches U2.15 (PA5)
- net TGT_SWCLK: now also J3.4 (Pin_4), U2.26 (PB13)
- net ~TGT_RESET: now reaches U2.18 (PB0)
- net ~TGT_RESET: now also J3.10 (Pin_10)
- net at U2.2 (PC13): now also R7.1
- net at U2.25 (PB12): now also R3.1
- net TGT_SWDIO: now reaches U2.27 (PB14)
- net TGT_SWDIO: now also J3.2 (Pin_2), R3.2
- net at U2.30 (PA9): now also R8.2
- net TGT_SWO: now reaches U2.31 (PA10)
- net TGT_SWO: now also J3.6 (Pin_6)
- net USB_DM: now reaches U2.32 (PA11)
- net USB_DM: now also R1.1
- net USB_DP: now reaches U2.33 (PA12)
- net USB_DP: now also R2.2
- net at U2.41 (PB5): now also R4.1
- net at U2.42 (PB6): now also R5.2
- net at U2.44 (BOOT0): now also R6.1
- net at U2.5 (PD0): now also C9.2, Y1.1
- net at U2.6 (PD1): now also C10.1, Y1.3
- net +5V: now reaches J1.A4 (VBUS), J1.A9 (VBUS), J1.B4 (VBUS), J1.B9 (VBUS)
- net +5V: now also C1.1, C2.1, U1.1 (VIN), U1.3 (EN)
- net at J1.A6 (D+): now also J1.B6 (D+), R2.1
- net at J1.A7 (D-): now also J1.B7 (D-), R1.2
- new net: D3.2 (A), R8.1
- new net: D1.1 (K), R4.2
- new net: D2.1 (K), R5.1
- no-connect marks 4 -> 25
Other:
- moved on the sheet: J1, J3, U2
